File: FritzenLab-egg-timer.kicad_pcb (KiCad board)
At the start: 2 copper layers, 14 parts, among them J1 Conn_01x05_Pin, J2 Conn_01x05_Pin, Q1 BC848, SW1 SW_Push_Dual, SW2 SW_Push_Dual, U1 PIC12F675-xSN

Commit message: almost finished PCB layout
Parts:
- moved R4 42.5 mm to (93.1, 65.9), turned to -90 degrees
- moved R5 35.7 mm to (82.6, 41.3)
- moved Q1 35.7 mm to (82.6, 44.2)
- moved BZ1 32.8 mm to (70.5, 47.9)
- moved R3 30.2 mm to (79.6, 66.0), turned to -90 degrees
- moved R1 22.9 mm to (73.8, 56.2)
- moved SW2 20.3 mm to (83.8, 65.8), turned to 180 degrees
- moved D1 18.4 mm to (75.3, 61.0), turned to 180 degrees
- moved SW1 18.1 mm to (97.3, 65.7), turned to 180 degrees
- moved C1 16.1 mm to (89.4, 42.2)
- moved R2 16.1 mm to (94.3, 44.1)
- moved U1 16.1 mm to (89.2, 46.2)
- moved J2 15.8 mm to (98.1, 41.7)
- moved J1 10.8 mm to (89.7, 37.8), turned to -90 degrees
Connections:
- SW1 pad 1: unconnected-(SW1-Pad1) -> Net-(R4-Pad2)
- SW1 pad 2: unconnected-(SW1-Pad2) -> Analog
- SW2 pad 1: unconnected-(SW2-Pad1) -> Net-(R3-Pad2)
- SW2 pad 2: unconnected-(SW2-Pad2) -> Analog
Routing:
- net VCC: track 0.00 -> 68.5 mm
- net Analog: track 0.00 -> 44.7 mm, vias 0 -> 2
- net LED: track 0.00 -> 16.6 mm, vias 0 -> 2
- net MCLR: track 0.00 -> 15.0 mm, vias 0 -> 1
- net Buzzer: track 0.00 -> 13.9 mm, vias 0 -> 2
- net PGC: track 0.00 -> 8.54 mm
- net Net-(BZ1--): track 0.00 -> 7.17 mm, vias 0 -> 1
- net GND: track 0.00 -> 6.72 mm, vias 0 -> 3
- net Net-(R4-Pad2): track 0.00 -> 6.29 mm
- net Net-(R3-Pad2): track 0.00 -> 6.29 mm
- net Net-(Q1-B): track 0.00 -> 5.15 mm
- net Net-(D1-A): track 0.00 -> 4.82 mm
- added copper zone on B.Cu, net GND
Other:
- board outline added: 34.5 x 34.5 mm
- board text added: "Egg timer 15/30/45/60 min"
- board text added: "FritzenLab.net"
- board text added: "Start"
- board text added: "Stop/reset"
