File: FritzenLab-egg-timer.kicad_sch (KiCad schematic)
At the start: 9 parts, among them J1 USB_B_Micro, Q1 BC848, SW1 SW_Push_Dual, SW2 SW_Push_Dual, U1 PIC12F675-xSN

Commit message: created PCB but not finished
Parts:
- removed J1: USB_B_Micro, Connector_USB:USB_Micro-B_Wuerth_629105150521, symbol Connector:USB_B_Micro
- added J1, J2: Conn_01x05_Pin, Connector_PinHeader_2.54mm:PinHeader_1x05_P2.54mm_Vertical, symbol Connector:Conn_01x05_Pin
- added R2, R3: 47k, Resistor_SMD:R_0805_2012Metric, symbol Device:R
- added R4: 68k, Resistor_SMD:R_0805_2012Metric, symbol Device:R
- added R5: 470, Resistor_SMD:R_0805_2012Metric, symbol Device:R
- BZ1: footprint (none) -> Buzzer_Beeper:Buzzer_12x9.5RM7.6
- C1: value C -> 100n; footprint (none) -> Capacitor_SMD:C_0805_2012Metric
- D1: footprint (none) -> LED_THT:LED_D5.0mm
- R1: value R -> 1k; footprint (none) -> Resistor_SMD:R_0805_2012Metric
- SW1, SW2: footprint (none) -> Button_Switch_SMD:SW_SPST_PTS810
Connections:
- net at SW1.3: now also R4.2
- net Analog: now reaches SW1.4
- net Analog: now also SW2.4, U1.7 (GP0), J2.4 (Pin_4), R2.1
- net VCC: now reaches U1.1 (VDD)
- net VCC: now also BZ1.1 (+), C1.1, J1.1 (Pin_1), J2.2 (Pin_2), R3.1, R4.1
- net LED: now reaches U1.2 (GP5)
- net LED: now also R1.1
- net MCLR: now reaches U1.4 (GP3)
- net MCLR: now also J2.1 (Pin_1)
- net Buzzer: now reaches U1.5 (GP2)
- net Buzzer: now also R5.1
- net PGC: now reaches U1.6 (GP1)
- net PGC: now also J2.5 (Pin_5)
- net GND: now reaches U1.8 (VSS)
- net GND: now also C1.2, D1.1 (K), Q1.2 (E), J1.5 (Pin_5), J2.3 (Pin_3), R2.2
- net at R1.2: now also D1.2 (A)
- net at SW2.3: now also R3.2
- net at Q1.1 (B): now also R5.2
- net at Q1.3 (C): now also BZ1.2 (-)

Commit message: almost finished PCB layout
Connections:
- net Analog: now also SW1.2, SW2.2; no longer SW1.4, SW2.4
- net at SW1.1: now also R4.2
- net at SW1.3: no longer R4.2
- net at SW2.1: now also R3.2
- net at SW2.3: no longer R3.2
Changed lines of the file:
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@@
 	(paper "A4")
 	(junction
-		(at 138.43 52.07)
+		(at 138.43 46.99)
 		(diameter 0)
 		(color 0 0 0 0)
-	)
-	(wire
-		(pts
-			(xy 119.38 52.07) (xy 124.46 52.07)
-		)
-		(stroke
-			(width 0)
-			(type default)
-		)
 	)
 	(wire
@@
 	(wire
 		(pts
+			(xy 138.43 29.21) (xy 138.43 46.99)
+		)
+		(stroke
+			(width 0)
+			(type default)
+		)
+	)
+	(wire
+		(pts
+			(xy 119.38 29.21) (xy 119.38 34.29)
+		)
+		(stroke
+			(width 0)
+			(type default)
+		)
+	)
+	(wire
+		(pts
 			(xy 172.72 44.45) (xy 172.72 52.07)
 		)
@@
 	(wire
 		(pts
-			(xy 134.62 34.29) (xy 138.43 34.29)
+			(xy 119.38 46.99) (xy 119.38 52.07)
 		)
 		(stroke
@@
 	(wire
 		(pts
-			(xy 138.43 34.29) (xy 138.43 52.07)
+			(xy 134.62 29.21) (xy 138.43 29.21)
 		)
 		(stroke
@@
 	(wire
 		(pts
-			(xy 138.43 52.07) (xy 138.43 55.88)
+			(xy 124.46 46.99) (xy 119.38 46.99)
 		)
 		(stroke
@@
 	(wire
 		(pts
-			(xy 134.62 52.07) (xy 138.43 52.07)
+			(xy 124.46 29.21) (xy 119.38 29.21)
 		)
 		(stroke
@@
 	(wire
 		(pts
-			(xy 119.38 34.29) (xy 124.46 34.29)
+			(xy 134.62 46.99) (xy 138.43 46.99)
 		)
 		(stroke
+			(width 0)
+			(type default)
+		)
+	)
+	(wire
+		(pts
+			(xy 138.43 46.99) (xy 138.43 55.88)
+		)
+		(stroke
